Commit message: add baxter init pose, add light

File: tsn_sim/urdf/ur5_robot.urdf.xacro (robot description, xacro)
@@ -12,5 +12,5 @@
     <parent link="world" />
     <child link = "base_link" />
-    <origin xyz="-0.5 0.0 1.1" rpy="0.0 0.0 0.0" />
+    <origin xyz="0.0 0.0 0.0" rpy="0.0 0.0 0.0" />
   </joint>
 </robot>
